File: ipradio.kicad_pcb (KiCad board)
At the start: 2 copper layers, 89 parts, among them IC1 AP2112K-3.3TRG1, IC2 CH224K, IC3 ESP32-C3, IC4 W25Q32RVXHJQ_TR, IC6 CP2102-GM, IC7 UDA1334BTS_N2,112, IC8 MP1584EN, J1 SJ-3524-SMT-TR, J2 USB4940-00-A, Q1 SS8050-G, Q2 SS8050-G, U1 2.42OLED, Y1 CM7V-T1A-32.768KHZ-7PF-20PPM-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, Y2 ABM8-40.000MHZ-10-1-U-T

Commit message: finalized schema
Parts:
- removed 2C5, C1, C2: 1uF, Capacitor_SMD:C_0402_1005Metric
- removed 2R9: 1k, Resistor_SMD:R_0402_1005Metric
- removed AE1: Antenna_Loop, ipradio:2.4_antenna_TI
- removed IC1: AP2112K-3.3TRG1, ipradio:SOT95P285X140-5N
- removed R24: 100k, Resistor_SMD:R_0402_1005Metric
- added 2C27: 1uF, Capacitor_SMD:C_1206_3216Metric, F.Cu at (90.2, 163.4)
- added 2C28: 100nF, Capacitor_SMD:C_1206_3216Metric, F.Cu at (87.8, 163.4)
- added 2C29: 10uF, Capacitor_SMD:C_1206_3216Metric, F.Cu at (85.4, 163.4)
- added 2C6: 10uF, Capacitor_SMD:C_0805_2012Metric, F.Cu at (118.4, 164.8)
- added 2C7: 1uF, Capacitor_SMD:C_0805_2012Metric, F.Cu at (116.3, 164.8)
- added 2C8: 100nF, Capacitor_SMD:C_0805_2012Metric, F.Cu at (114.3, 164.8)
- added 2R12: 10k, Resistor_SMD:R_0402_1005Metric, F.Cu at (75.7, 170.7)
- added 3C19: 100nF, Capacitor_SMD:C_0402_1005Metric, F.Cu at (172.2, 151.9)
- added 3C20: 1uF, Capacitor_SMD:C_0402_1005Metric, F.Cu at (172.2, 153.9)
- added 3C21: 10uF, Capacitor_SMD:C_0402_1005Metric, F.Cu at (172.2, 155.8)
- added 3FB1: 100mHz, Inductor_SMD:L_0402_1005Metric, F.Cu at (151.8, 154.1)
- added 4C11: 1uF, Capacitor_SMD:C_0402_1005Metric, F.Cu at (61.7, 61.3)
- added 4C12: 100nF, Capacitor_SMD:C_0402_1005Metric, F.Cu at (61.7, 63.3)
- added 4C13: 100nF, Capacitor_SMD:C_0402_1005Metric, F.Cu at (61.7, 65.2)
- added 4C17: 1uF, Capacitor_SMD:C_0402_1005Metric, F.Cu at (172.2, 157.8)
- added 4C18: 100nF, Capacitor_SMD:C_0402_1005Metric, F.Cu at (172.2, 159.8)
- added 4FB1: 100mHz, Inductor_SMD:L_0402_1005Metric, F.Cu at (64.6, 58.3)
- added 4R10: 10k, Resistor_SMD:R_0402_1005Metric, F.Cu at (70.4, 62.3)
- added 4R11: 10k, Resistor_SMD:R_0402_1005Metric, F.Cu at (70.4, 64.3)
- added 4R5: 5.1k, Resistor_SMD:R_0402_1005Metric, F.Cu at (67.5, 60.3)
- added 4R9: 10k, Resistor_SMD:R_0402_1005Metric, F.Cu at (70.4, 60.3)
- added 5C3: 100nF, Capacitor_SMD:C_0402_1005Metric, F.Cu at (275.5, 143.6)
- added 5C4: 100nF, Capacitor_SMD:C_0402_1005Metric, F.Cu at (158.6, 79.3)
- added 5C5: 1uF, Capacitor_SMD:C_0402_1005Metric, F.Cu at (158.6, 81.2)
- added 5C6: 10uF, Capacitor_SMD:C_0402_1005Metric, F.Cu at (158.6, 83.2)
- added 5C7: 100nF, Capacitor_SMD:C_0402_1005Metric, F.Cu at (152.6, 51.8)
- added C19: 1uF, Capacitor_SMD:C_0402_1005Metric, F.Cu at (236.8, 113.2)
- added C20: 1uF, Capacitor_SMD:C_0402_1005Metric, F.Cu at (232.2, 115.7)
- added IC10: SPX1117M3-L-3-3_TR, ipradio:SOT230P700X180-4N, F.Cu at (163.9, 157.3)
- added IC5: NJM2882F33-TE1, ipradio:SOT95P280X130-5N, F.Cu at (65.8, 67.6)
- added J4: CONMHF1-SMD-T, ipradio:CONMHF1SMDT, F.Cu at (231.8, 96.3)
- added R1: 10k, Resistor_SMD:R_0402_1005Metric, F.Cu at (234.2, 115.7)
- added R2: 5.1k, Resistor_SMD:R_0402_1005Metric, F.Cu at (149.7, 49.9)
- added R3: 5.1k, Resistor_SMD:R_0402_1005Metric, F.Cu at (149.7, 51.9)
- added R4: 5.1k, Resistor_SMD:R_0402_1005Metric, F.Cu at (272.6, 153.6)
- added U2: SMS-202C, ipradio:SMS202F, F.Cu at (233.4, 109.2)
- 2D2, 2D3: value SS34 -> D_TVS; footprint ipradio:DIOM7959X265N -> Diode_SMD:D_SOD-123
- 2R11: value 10k -> 1k
- C15, C17: value 0.1uF -> 100nF
- moved J1 234.2 mm to (36.4, 51.0)
- moved 4C1 183.4 mm to (61.7, 51.5)
- moved 4C10 183.4 mm to (61.7, 59.3)
- moved 4C2 183.4 mm to (61.7, 53.4)
- moved 4C6 183.4 mm to (61.7, 55.4)
- moved 4C8 183.4 mm to (61.7, 57.4)
- moved 4C3 180.6 mm to (57.3, 52.6)
- moved 4C4 180.6 mm to (57.3, 57.0)
- moved 4C5 180.6 mm to (57.3, 61.4)
- moved 4C7 180.6 mm to (57.3, 65.7)
- moved 4C9 180.6 mm to (57.3, 70.0)
- moved IC7 180.4 mm to (67.6, 53.9)
- moved 4R1 176.6 mm to (64.6, 60.3)
- moved 4R2 176.6 mm to (64.6, 62.3)
- moved 4R3 176.6 mm to (64.6, 64.3)
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Connections:
- net OLED_MOSI renamed I2S_SDA
- 2C2 pad 1: Net-(2C2-Pad1) -> V_SYS_5V2A
- 2C26 pad 1: VBUS_9V -> VBUS_5V3A_9V1.5A
- 2L1 pad 1: Net-(2C2-Pad1) -> V_SYS_5V2A
- 2R1 pad 1: Net-(2C2-Pad1) -> V_SYS_5V2A
- 2R11 pad 1: Net-(IC2-VBUS) -> VBUS_5V3A_9V1.5A
- 2R11 pad 2: VBUS_9V -> Net-(IC2-VDD)
- 2R16 pad 2: Net-(IC2-CC1) -> /power_supply/CC1
- 2R17 pad 2: Net-(IC2-CC2) -> /power_supply/CC2
- 2R5 pad 1: VBUS_9V -> VBUS_5V3A_9V1.5A
- 2R5 pad 2: /power_supply/EN -> Net-(IC8-EN)
- 2R6 pad 2: /power_supply/EN -> VBUS_5V3A_9V1.5A
- 2R7 pad 1: Net-(IC2-CFG1) -> GND
- 2R7 pad 2: GND -> Net-(IC2-CFG1)
- 4C1 pad 2: GND -> GNDA
- 4C10 pad 2: GND -> GNDA
- 4C2 pad 2: GND -> GNDA
- 4C7 pad 2: GND -> GNDA
- 4C8 pad 2: GND -> GNDA
- 4C9 pad 2: GND -> GNDA
- 4R1 pad 2: GND -> GNDA
- 4R2 pad 2: GND -> GNDA
- 4R6 pad 1: +3V3 -> 3V3
- 4R7 pad 1: +3V3 -> VDDA3V3
- 4R8 pad 1: GND -> GNDA
- 5R1 pad 1: ENC_E1 -> 3V3
- 5R1 pad 2: Net-(S3-S2) -> ENC_CLK
- 5R2 pad 1: ENC_D1 -> 3V3
- 5R2 pad 2: Net-(S3-S1) -> ENC_DT
- 5R3 pad 1: +3V3 -> Net-(U1-RES)
- 5R3 pad 2: Net-(U1-RES) -> 3V3
- C11 pad 1: +3V3 -> 3V3
- C13 pad 1: Net-(S2-COM_1) -> /esp32/EN
- C15 pad 1: +3V3 -> 3V3
- C16 pad 1: GND -> /esp32/XTAL_N
- C16 pad 2: /esp32/XTAL_N -> GND
- C17 pad 1: +3V3 -> 3V3
- C23 pad 1: +3V3 -> 3V3
- C24 pad 1: +3V3 -> 3V3
- C6 pad 1: +3V3 -> 3V3
- C7 pad 1: +3V3 -> 3V3
- C9 pad 1: +3V3 -> 3V3
- IC2 pad 1: VDD -> Net-(IC2-VDD)
- IC2 pad 6: Net-(IC2-CC2) -> /power_supply/CC2
- IC2 pad 7: Net-(IC2-CC1) -> /power_supply/CC1
- IC3 pad 11: +3V3 -> 3V3
- IC3 pad 13: I2S_MCLK -> I2S_CLK
- IC3 pad 14: OLED_CLK -> /esp32/GPIO8
- IC3 pad 17: +3V3 -> 3V3
- IC3 pad 25: OLED_DC -> ENC_DT
- IC3 pad 26: OLED_CS -> ENC_CLK
- IC3 pad 31: +3V3 -> 3V3
- IC3 pad 32: +3V3 -> 3V3
- IC3 pad 6: ENC_E1 -> ENC_SW
- IC3 pad 8: ENC_D1 -> /esp32/GPIO3
- IC6 pad 2: GND -> unconnected-(IC6-RI-Pad2)
- IC6 pad 6: +3V3 -> 3V3
- IC6 pad 7: +3V3 -> 3V3
- IC7 pad 10: GND -> unconnected-(IC7-PCS-Pad10)
- IC7 pad 11: GND -> Net-(IC7-SFOR0)
- IC7 pad 15: GND -> GNDA
- IC7 pad 6: I2S_MCLK -> unconnected-(IC7-SYSCLK-Pad6)
- IC7 pad 7: GND -> Net-(IC7-SFOR1)
- IC7 pad 9: GND -> Net-(IC7-DEEM)
- IC8 pad 2: /power_supply/EN -> Net-(IC8-EN)
- IC8 pad 7: VBUS_9V -> VBUS_5V3A_9V1.5A
- J1 pad 1: GND -> GNDA
- J2 pad A4: VBUS_9V -> VBUS_5V3A_9V1.5A
- J2 pad A5: Net-(IC2-CC1) -> /power_supply/CC1
- J2 pad B4: VBUS_9V -> VBUS_5V3A_9V1.5A
- J2 pad B5: Net-(IC2-CC2) -> /power_supply/CC2
- L2 pad 1: +3V3 -> 3V3
- R14 pad 1: +3V3 -> 3V3
- R14 pad 2: Net-(S2-COM_1) -> /esp32/EN
- R15 pad 2: +3V3 -> 3V3
- R19 pad 1: +5V_BUS -> V_SYS_5V2A
- R22 pad 1: +3V3 -> 3V3
- S1 pad 1: /esp32/GPIO9 -> GND
- S1 pad 2: /esp32/GPIO9 -> GND
- S1 pad 3: GND -> /esp32/GPIO9
- S1 pad 4: GND -> /esp32/GPIO9
- S2 pad 1: Net-(S2-COM_1) -> /esp32/EN
- S2 pad 2: Net-(S2-COM_1) -> /esp32/EN
- S3 pad A1: unconnected-(S3-NO_1-PadA1) -> ENC_DT
- S3 pad B1: unconnected-(S3-NO_2-PadB1) -> ENC_CLK
- S3 pad D1: Net-(S3-S1) -> ENC_SW
- S3 pad E1: Net-(S3-S2) -> ENC_SW
- U1 pad 2: +3V3 -> 3V3
- U1 pad 3: OLED_CLK -> I2S_CLK
- U1 pad 6: OLED_DC -> unconnected-(U1-DC-Pad6)
- U1 pad 7: OLED_CS -> unconnected-(U1-CS-Pad7)

Commit message: pcb for power and esp32
Parts:
- removed C21, C22: 10pF, Capacitor_SMD:C_0402_1005Metric
- removed R21: 10МОм, Resistor_SMD:R_0402_1005Metric
- removed Y1: CM7V-T1A-32.768KHZ-7PF-20PPM-TA-QC, ipradio:CM7V32768TBQA020
- 2R5: value 91k -> 100k
- 2R6: value 24.9k -> 24k
- S1, S2, S3, U1: moved to B.Cu
- moved 2R16 117.2 mm to (130.7, 67.7), turned to -90 degrees
- moved 2R12 117.1 mm to (137.0, 70.9), turned to 90 degrees
- moved 2D2 116.2 mm to (132.4, 66.6)
- moved 2R7 116.0 mm to (138.1, 70.9), turned to 90 degrees
- moved IC2 115.8 mm to (137.0, 66.2)
- moved 2R17 115.5 mm to (130.7, 72.0)
- moved J2 114.7 mm to (124.9, 69.6)
- moved 2D3 112.5 mm to (132.4, 73.3), turned to 90 degrees
- moved 2R11 112.2 mm to (140.3, 66.2), turned to 90 degrees
- moved 2R6 111.1 mm to (150.8, 63.3)
- moved 2R1 110.8 mm to (144.2, 65.6)
- moved 2C3 110.6 mm to (148.5, 63.3)
- moved IC8 110.6 mm to (149.1, 68.0)
- moved 2R3 110.6 mm to (147.2, 63.2)
- moved 2R4 110.6 mm to (148.0, 72.6)
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Connections:
- IC3 pad 26: ENC_CLK -> /esp32/GPIO19
- IC3 pad 8: /esp32/GPIO3 -> ENC_CLK
Routing:
- net 3V3: track 0.00 -> 98.6 mm, vias 0 -> 4
- net /esp32/TX: track 0.00 -> 73.8 mm, vias 0 -> 2
- net /esp32/RX: track 0.00 -> 70.6 mm, vias 0 -> 2
- net /esp32/GPIO9: track 0.00 -> 67.3 mm, vias 0 -> 3
- net USB_DP: track 0.00 -> 67.2 mm, vias 0 -> 2
- net USB_DN: track 0.00 -> 63.4 mm, vias 0 -> 1
- net /esp32/EN: track 0.00 -> 58.3 mm, vias 0 -> 3
- net VBUS_5V3A_9V1.5A: track 0.00 -> 25.6 mm, vias 0 -> 5
- net V_SYS_5V2A: track 0.00 -> 23.1 mm, vias 0 -> 2
- net /esp32/XTAL_N: track 0.00 -> 11.4 mm
- net /esp32/RTS: track 0.00 -> 9.87 mm
- net Net-(IC3-VDD3P3_1): track 0.00 -> 9.25 mm
- net /power_supply/CC2: track 0.00 -> 9.12 mm
- net /power_supply/CC1: track 0.00 -> 8.42 mm
- net Net-(Q2-B): track 0.00 -> 7.94 mm
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- added copper zone on F.Cu, net 3V3
- added copper zone on B.Cu, net GND
- added copper zone on F.Cu, net GND
- added copper zone on In1.Cu, net GND
- added copper zone on In2.Cu, net GND
- added copper zone on F.Cu, net Net-(IC10-VIN)
- added copper zone on F.Cu, net Net-(IC8-FB)
- added copper zone on F.Cu, net Net-(IC8-SW)
- added copper zone on F.Cu, net VBUS_5V3A_9V1.5A
- added copper zone on F.Cu, net V_SYS_5V2A
Other:
- board outline added: 95.7 x 53.5 mm
- copper layers 2 -> 4

Commit message: pcb for power and esp32
Routing:
- removed copper zone on B.Cu, net GND
- removed copper zone on F.Cu, net GND
- removed copper zone on In1.Cu, net GND
- removed copper zone on In2.Cu, net GND
Changed lines of the file:
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@@
 		(capping no)
 		(filling no)
-		(zone_defaults)
 		(pcbplotparams
 			(layerselection 0x00000000_00000000_55555555_5755f5ff)
@@
 	)
 	(segment
-		(start 207.2 60.733273)
-		(end 207.2 60.75)
-		(width 0.15)
-		(layer "F.Cu")
-		(net "/esp32/GPIO9")
-	)
-	(segment
-		(start 178.7 60.15)
-		(end 179.61 60.15)
-		(width 0.254)
-		(layer "F.Cu")
-		(net "/esp32/GPIO9")
-	)
-	(segment
-		(start 179.61 60.15)
-		(end 179.7 60.06)
-		(width 0.254)
-		(layer "F.Cu")
-		(net "/esp32/GPIO9")
-	)
-	(segment
-		(start 205.75 58.749999)
-		(end 205.75 59.283273)
-		(width 0.15)
-		(layer "F.Cu")
-		(net "/esp32/GPIO9")
-	)
-	(segment
-		(start 205.75 59.283273)
-		(end 207.2 60.733273)
-		(width 0.15)
-		(layer "F.Cu")
-		(net "/esp32/GPIO9")
-	)
-	(via
-		(at 178.7 83.55)
-		(size 0.6)
-		(drill 0.3)
-		(layers "F.Cu" "B.Cu")
-		(net "/esp32/GPIO9")
-	)
-	(via
-		(at 178.7 60.15)
-		(size 0.6)
-		(drill 0.3)
-		(layers "F.Cu" "B.Cu")
-		(net "/esp32/GPIO9")
-	)
-	(via
-		(at 207.2 60.75)
-		(size 0.6)
-		(drill 0.3)
-		(layers "F.Cu" "B.Cu")
-		(net "/esp32/GPIO9")
-	)
-	(segment
-		(start 202.65 56.2)
-		(end 207.2 60.75)
-		(width 0.254)
-		(layer "B.Cu")
-		(net "/esp32/GPIO9")
-	)
-	(segment
-		(start 178.7 83.55)
-		(end 170.5 83.55)
-		(width 0.254)
-		(layer "B.Cu")
-		(net "/esp32/GPIO9")
-	)
-	(segment
-		(start 182.609 56.241)
-		(end 200.842998 56.241)
-		(width 0.254)
-		(layer "B.Cu")
-		(net "/esp32/GPIO9")
-	)
-	(segment
-		(start 178.7 60.15)
-		(end 178.7 83.55)
-		(width 0.254)
-		(layer "B.Cu")
-		(net "/esp32/GPIO9")
-	)
-	(segment
-		(start 200.883998 56.2)
-		(end 202.65 56.2)
-		(width 0.254)
-		(layer "B.Cu")
-		(net "/esp32/GPIO9")
-	)
-	(segment
-		(start 200.842998 56.241)
-		(end 200.883998 56.2)
-		(width 0.254)
-		(layer "B.Cu")
-		(net "/esp32/GPIO9")
-	)
-	(segment
-		(start 178.7 60.15)
-		(end 182.609 56.241)
-		(width 0.254)
-		(layer "B.Cu")
-		(net "/esp32/GPIO9")
-	)
-	(segment
 		(start 178.35 64.35)
 		(end 179.32 64.35)
@@
 	)
 	(segment
+		(start 207.2 60.733273)
+		(end 207.2 60.75)
+		(width 0.15)
+		(layer "F.Cu")
+		(net "/esp32/GPIO9")
+	)
+	(segment
+		(start 178.7 60.15)
+		(end 179.61 60.15)
+		(width 0.254)
+		(layer "F.Cu")
+		(net "/esp32/GPIO9")
+	)
+	(segment
+		(start 179.61 60.15)
+		(end 179.7 60.06)
+		(width 0.254)
+		(layer "F.Cu")
+		(net "/esp32/GPIO9")
+	)
+	(segment
+		(start 205.75 58.749999)
+		(end 205.75 59.283273)
+		(width 0.15)
+		(layer "F.Cu")
+		(net "/esp32/GPIO9")
+	)
+	(segment
+		(start 205.75 59.283273)
+		(end 207.2 60.733273)
+		(width 0.15)
+		(layer "F.Cu")
+		(net "/esp32/GPIO9")
+	)
+	(via
+		(at 178.7 83.55)
+		(size 0.6)
+		(drill 0.3)
+		(layers "F.Cu" "B.Cu")
+		(net "/esp32/GPIO9")
+	)
+	(via
+		(at 178.7 60.15)
+		(size 0.6)
+		(drill 0.3)
+		(layers "F.Cu" "B.Cu")
+		(net "/esp32/GPIO9")
+	)
+	(via
+		(at 207.2 60.75)
+		(size 0.6)
+		(drill 0.3)
+		(layers "F.Cu" "B.Cu")
+		(net "/esp32/GPIO9")
+	)
+	(segment
+		(start 202.65 56.2)
+		(end 207.2 60.75)
+		(width 0.254)
+		(layer "B.Cu")
+		(net "/esp32/GPIO9")
+	)
+	(segment
+		(start 178.7 83.55)
+		(end 170.5 83.55)
+		(width 0.254)
+		(layer "B.Cu")
+		(net "/esp32/GPIO9")
+	)
+	(segment
+		(start 182.609 56.241)
+		(end 200.842998 56.241)
+		(width 0.254)
+		(layer "B.Cu")
+		(net "/esp32/GPIO9")
+	)
+	(segment
+		(start 178.7 60.15)
+		(end 178.7 83.55)
+		(width 0.254)
+		(layer "B.Cu")
+		(net "/esp32/GPIO9")
+	)
+	(segment
+		(start 200.883998 56.2)
+		(end 202.65 56.2)
+		(width 0.254)
+		(layer "B.Cu")
+		(net "/esp32/GPIO9")
+	)
+	(segment
+		(start 200.842998 56.241)
+		(end 200.883998 56.2)
+		(width 0.254)
+		(layer "B.Cu")
+		(net "/esp32/GPIO9")
+	)
+	(segment
+		(start 178.7 60.15)
+		(end 182.609 56.241)
+		(width 0.254)
+		(layer "B.Cu")
+		(net "/esp32/GPIO9")
+	)
+	(segment
 		(start 208.392306 57.373044)
 		(end 208.609631 57.590369)
@@
 		(layer "F.Cu")
 		(hatch edge 0.5)
-		(priority 2)
+		(priority 3)
 		(connect_pads yes
 			(clearance 0.5)
@@
 		(layer "F.Cu")
 		(hatch edge 0.5)
-		(priority 1)
+		(priority 2)
 		(connect_pads yes
 			(clearance 0.5)
@@
 		(layer "F.Cu")
 		(hatch edge 0.5)
-		(priority 5)
+		(priority 6)
 		(connect_pads yes
 			(clearance 0.5)
@@
 		(layer "F.Cu")
 		(hatch edge 0.5)
-		(priority 6)
+		(priority 7)
 		(connect_pads yes
 			(clearance 0.5)
@@
 		(layer "F.Cu")
 		(hatch edge 0.5)
+		(priority 1)
 		(connect_pads yes
 			(clearance 0.5)
@@
 		(layer "F.Cu")
 		(hatch edge 0.5)
-		(priority 4)
+		(priority 5)
 		(connect_pads yes
 			(clearance 0.5)
@@
 		(layer "F.Cu")
 		(hatch edge 0.5)
-		(priority 3)
+		(priority 4)
 		(connect_pads yes
 			(clearance 0.5)
@@
 		(layer "F.Cu")
 		(hatch edge 0.5)
-		(priority 8)
+		(priority 9)
 		(connect_pads yes
 			(clearance 0.5)
@@
 		(layer "F.Cu")
 		(hatch edge 0.5)
-		(priority 7)
+		(priority 8)
 		(connect_pads yes
 			(clearance 0.5)
@@
 			)
 		)
-	)
-	(zone
-		(net "GND")
-		(layers "F.Cu" "B.Cu" "In1.Cu" "In2.Cu")
-		(hatch edge 0.5)
-		(priority 9)
-		(connect_pads yes
-			(clearance 0.5)
-		)
-		(min_thickness 0.25)
-		(fill yes
-			(thermal_gap 0.5)
-			(thermal_bridge_width 0.5)
-			(island_removal_mode 0)
-		)
-		(polygon
-			(pts
-				(xy 119.6 58.8) (xy 163.95 58.85) (xy 163.95 54.95) (xy 194.9 54.95) (xy 194.9 37.75) (xy 214.95 37.85)
-				(xy 215.2 90.2) (xy 119.9 89.95) (xy 119.75 58.65)
-			)
-		)
